Commit message: added navigation

File: verter_admin/src/verter_admin/urdf/verter_robot_gazebo.urdf (robot description, URDF)
Before this commit: robot verter_robot, 14 links, 13 joints
Links:
- removed link camera_tof
- removed link camera_tof_optical
- added link imu_link, mass 0.001; collision box size=0.02 0.02 0.01; visual box size=0.02 0.02 0.01
- added link lidar_link, mass 0.190; collision cylinder length=0.04 radius=0.038; visual cylinder length=0.04 radius=0.038
- link wheel_left: mass 2.0 -> 0.8
- link wheel_right: mass 2.0 -> 0.8
Joints:
- removed joint camera_tof_joint
- removed joint camera_tof_optical_joint
- added joint imu_joint: type fixed, parent base_link, child imu_link, origin xyz=0 0 0.05 rpy=0 0 0
- added joint lidar_joint: type fixed, parent base_link, child lidar_link, origin xyz=0.28 0 0.70 rpy=0 0 0
