Commit message: added nav2 + slam

File: verter_admin/src/verter_admin/urdf/verter_robot_minimal.urdf (robot description, URDF)
Before this commit: robot verter_robot, 12 links, 11 joints
Links:
- link base_link: geometry collision box size=0.580 0.554 0.550; visual box size=0.560 0.534 0.550
Joints:
- joint caster_back_joint: origin xyz=-0.12 0 -0.07 rpy=0 0 0 -> xyz=-0.22 0 -0.07 rpy=0 0 0
- joint sensor_front_center_joint: origin xyz=0.16 0 0.08 rpy=0 0 0 -> xyz=0.280 0 0.048 rpy=0 0 0
- joint sensor_front_left_inner_joint: origin xyz=0.15 0.05 0.08 rpy=0 0 0.4363 -> xyz=0.260 0.08 0.048 rpy=0 0 0.4363
- joint sensor_front_left_outer_joint: origin xyz=0.14 0.10 0.08 rpy=0 0 0.7854 -> xyz=0.230 0.16 0.048 rpy=0 0 0.7854
- joint sensor_front_right_inner_joint: origin xyz=0.15 -0.05 0.08 rpy=0 0 -0.4363 -> xyz=0.260 -0.08 0.048 rpy=0 0 -0.4363
- joint sensor_front_right_outer_joint: origin xyz=0.14 -0.10 0.08 rpy=0 0 -0.7854 -> xyz=0.230 -0.16 0.048 rpy=0 0 -0.7854
- joint sensor_left_joint: origin xyz=0 0.11 0.08 rpy=0 0 1.5708 -> xyz=0 0.267 0.048 rpy=0 0 1.5708
- joint sensor_right_joint: origin xyz=0 -0.11 0.08 rpy=0 0 -1.5708 -> xyz=0 -0.267 0.048 rpy=0 0 -1.5708
- joint wheel_left_joint: origin xyz=0.10 0.11 0 rpy=0 0 0 -> xyz=0.05 0.178 0 rpy=0 0 0
- joint wheel_right_joint: origin xyz=0.10 -0.11 0 rpy=0 0 0 -> xyz=0.05 -0.178 0 rpy=0 0 0

Commit message: added tof camera to navigation

File: verter_admin/src/verter_admin/urdf/verter_robot_minimal.urdf (robot description, URDF)
Before this commit: robot verter_robot, 12 links, 11 joints
Links:
- added link camera_tof; visual box size=0.03 0.06 0.02
- added link camera_tof_optical
Joints:
- added joint camera_tof_joint: type fixed, parent base_link, child camera_tof, origin xyz=0.150 0 0.400 rpy=0 0 0
- added joint camera_tof_optical_joint: type fixed, parent camera_tof, child camera_tof_optical, origin xyz=0 0 0 rpy=-1.5708 0 -1.5708
- joint sensor_front_left_inner_joint: origin xyz=0.260 0.08 0.048 rpy=0 0 0.4363 -> xyz=0.277 0.074 0.048 rpy=0 0 0.0995
- joint sensor_front_left_outer_joint: origin xyz=0.230 0.16 0.048 rpy=0 0 0.7854 -> xyz=0.262 0.152 0.048 rpy=0 0 0.2304
- joint sensor_front_right_inner_joint: origin xyz=0.260 -0.08 0.048 rpy=0 0 -0.4363 -> xyz=0.277 -0.074 0.048 rpy=0 0 -0.0995
- joint sensor_front_right_outer_joint: origin xyz=0.230 -0.16 0.048 rpy=0 0 -0.7854 -> xyz=0.262 -0.152 0.048 rpy=0 0 -0.2304
- joint sensor_left_joint: origin xyz=0 0.267 0.048 rpy=0 0 1.5708 -> xyz=0.180 0.228 0.048 rpy=0 0 1.3265
- joint sensor_right_joint: origin xyz=0 -0.267 0.048 rpy=0 0 -1.5708 -> xyz=0.180 -0.228 0.048 rpy=0 0 -1.3265
- joint wheel_left_joint: origin xyz=0.05 0.178 0 rpy=0 0 0 -> xyz=0.120 0.178 0 rpy=0 0 0
- joint wheel_right_joint: origin xyz=0.05 -0.178 0 rpy=0 0 0 -> xyz=0.120 -0.178 0 rpy=0 0 0

Commit message: added lidar to urdf

File: verter_admin/src/verter_admin/urdf/verter_robot_minimal.urdf (robot description, URDF)
Before this commit: robot verter_robot, 14 links, 13 joints
Links:
- added link lidar_link; visual cylinder length=0.04 radius=0.035
Joints:
- added joint lidar_joint: type fixed, parent base_link, child lidar_link, origin xyz=0.0 0 0.450 rpy=0 0 0

Commit message: updated moving and mapping flow

File: verter_admin/src/verter_admin/urdf/verter_robot_minimal.urdf (robot description, URDF)
Before this commit: robot verter_robot, 15 links, 14 joints
Links:
- removed link base_footprint
Joints:
- removed joint base_footprint_joint
- joint lidar_joint: origin xyz=0.0 0 0.450 rpy=0 0 0 -> xyz=0.25 0 0.450 rpy=0 0 0

Commit message: added calibration_node.py and some fixes

File: verter_admin/src/verter_admin/urdf/verter_robot_minimal.urdf (robot description, URDF)
Before this commit: robot verter_robot, 14 links, 13 joints
Links:
- added link base_footprint
Joints:
- added joint base_footprint_joint: type fixed, parent base_footprint, child base_link, origin xyz=0 0 0.1 rpy=0 0 0
- joint lidar_joint: origin xyz=0.25 0 0.450 rpy=0 0 0 -> xyz=0.12 0 0.70 rpy=0 0 0

Commit message: lidar shift

File: verter_admin/src/verter_admin/urdf/verter_robot_minimal.urdf (robot description, URDF)
Before this commit: robot verter_robot, 15 links, 14 joints
Joints:
- joint lidar_joint: origin xyz=0.12 0 0.70 rpy=0 0 0 -> xyz=0.12 0 0.70 rpy=0 0 3.14159

Commit message: added IMU and esp32

File: verter_admin/src/verter_admin/urdf/verter_robot_minimal.urdf (robot description, URDF)
Before this commit: robot verter_robot, 15 links, 14 joints
Links:
- added link imu_link; visual box size=0.03 0.03 0.01
Joints:
- added joint imu_joint: type fixed, parent base_link, child imu_link, origin xyz=0 0 0.29 rpy=0 0 0

Commit message: calibration

File: verter_admin/src/verter_admin/urdf/verter_robot_minimal.urdf (robot description, URDF)
Before this commit: robot verter_robot, 16 links, 15 joints
Joints:
- joint imu_joint: origin xyz=0 0 0.29 rpy=0 0 0 -> xyz=0.09 0 0.29 rpy=0 0 0

Commit message: added ultrasonic Range displays to rviz config

File: verter_admin/src/verter_admin/urdf/verter_robot_minimal.urdf (robot description, URDF)
Before this commit: robot verter_robot, 16 links, 15 joints
Joints:
- joint wheel_left_joint: axis 0 1 0 -> (none); type continuous -> fixed
- joint wheel_right_joint: axis 0 1 0 -> (none); type continuous -> fixed
