Commit message: System setup

File: verter_admin/src/verter_admin/urdf/verter_robot_minimal.urdf (robot description, URDF)
Before this commit: robot verter_robot, 16 links, 15 joints
Joints:
- joint imu_joint: origin xyz=0.09 0 0.29 rpy=0 0 0 -> xyz=0 0 0.305 rpy=0 0 0
- joint lidar_joint: origin xyz=0.12 0 0.70 rpy=0 0 3.14159 -> xyz=0 0 0.76 rpy=0 0 3.14159
- joint wheel_left_joint: origin xyz=0.120 0.178 0 rpy=0 0 0 -> xyz=0 0.178 0 rpy=0 0 0
- joint wheel_right_joint: origin xyz=0.120 -0.178 0 rpy=0 0 0 -> xyz=0 -0.178 0 rpy=0 0 0
